Commit message: added logic for lite gripper fingers

File: xarm_description/urdf/gripper/gripper_macro.xacro (robot description, xacro)
@@ -13,6 +13,6 @@
     <xacro:if value="${robot_type == 'lite'}">
       <!-- Load Lite Gripper Model URDF -->
-      <xacro:include filename="$(find xarm_description)/urdf/gripper/lite_gripper.urdf.xacro" />
-      <xacro:uflite_gripper_urdf prefix="${prefix}" />
+      <xacro:include filename="$(find xarm_description)/urdf/gripper/lite_gripper_macro.xacro" />
+      <xacro:lite_gripper_macro prefix="${prefix}" />
     </xacro:if>
     <xacro:if value="${robot_type == 'bio'}">

File: xarm_description/urdf/gripper/lite_gripper.urdf.xacro (robot description, xacro)
@@ -1,13 +1,15 @@
 <?xml version="1.0"?>
-<robot xmlns:xacro="http://ros.org/wiki/xacro" name="uflite_gripper">
-  <xacro:macro name="uflite_gripper_urdf" params="prefix:='' attach_to:='' attach_xyz:='0 0 0' attach_rpy:='0 0 0' ">
+<robot xmlns:xacro="http://ros.org/wiki/xacro" name="uf_lite_gripper">
+  <xacro:macro name="lite_gripper_urdf" params="prefix:='' attach_to:='' attach_xyz:='0 0 0' attach_rpy:='0 0 0' ">
+    <!-- Gripper Fix Joint -->
     <xacro:unless value="${attach_to == ''}">
       <joint name="${prefix}gripper_fix" type="fixed">
         <parent link="${attach_to}"/>
-        <child link="${prefix}uflite_gripper_link"/>
+        <child link="${prefix}lite_gripper_base_link"/>
         <origin xyz="${attach_xyz}" rpy="${attach_rpy}"/>
       </joint>
     </xacro:unless>
-    <link name="${prefix}uflite_gripper_link">
+    <!-- Base link of the gripper -->
+    <link name="${prefix}lite_gripper_base_link">
       <inertial>
         <origin xyz="0.0 0.0 0.030" rpy="0 0 0" />
@@ -18,17 +20,71 @@
       </inertial>
       <xacro:common_link_visual
-        mesh_filename="gripper/lite/visual/gripper_lite"
+        mesh_filename="gripper/lite/visual/gripper_lite_body"
         origin_xyz="0 0 0"
         origin_rpy="0 0 0"
         material_name="${prefix}White" />
       <xacro:common_link_collision
-        mesh_filename="gripper/lite/collision/gripper_lite"
+        mesh_filename="gripper/lite/collision/gripper_lite_body"
         origin_xyz="0 0 0"
         origin_rpy="0 0 0" />
     </link>
+    <!-- Left Finger -->
+    <link name="${prefix}lite_gripper_left_finger">
+      <inertial>
+        <origin xyz="0 0.0078 0.0543" rpy="0 0 0" />
+        <mass value="0.012105" />
+        <inertia
+          ixx="3.7322E-06" ixy="-4.1705E-06" ixz="4.0142E-06"
+          iyy="1.744E-05" iyz="-1.2237E-06" izz="1.7775E-05" />
+      </inertial>
+      <xacro:common_link_visual
+        mesh_filename="gripper/lite/visual/gripper_lite_finger"
+        origin_xyz="0 0.0078 0.0543"
+        origin_rpy="0 0 3.14159"
+        material_name="${prefix}White" />
+      <xacro:common_link_collision
+        mesh_filename="gripper/lite/collision/gripper_lite_finger"
+        origin_xyz="0 0.0078 0.0543"
+        origin_rpy="0 0 3.14159" />
+    </link>
+    <joint name="${prefix}left_finger_joint" type="prismatic">
+      <origin xyz="0 0 0" rpy="0 0 0"/>
+      <parent link="${prefix}lite_gripper_base_link"/>
+      <child link="${prefix}lite_gripper_left_finger"/>
+      <axis xyz="0 1 0"/>
+      <limit lower="0.0" upper="0.0081" effort="2" velocity="0.1"/>
+      <mimic joint="${prefix}right_finger_joint" multiplier="1" offset="0" />
+    </joint>
+    <!-- Right Finger -->
+    <link name="${prefix}lite_gripper_right_finger">
+      <inertial>
+        <origin xyz="0 -0.0078 0.0543" rpy="0 0 0" />
+        <mass value="0.012068" />
+        <inertia
+          ixx="4.1413E-06" ixy="3.9682E-06" ixz="4.5734E-06"
+          iyy="1.6115E-05" iyz="1.6711E-06" izz="1.6032E-05" />
+      </inertial>
+      <xacro:common_link_visual
+        mesh_filename="gripper/lite/visual/gripper_lite_finger"
+        origin_xyz="0 -0.0078 0.0543"
+        origin_rpy="0 0 0"
+        material_name="${prefix}White" />
+      <xacro:common_link_collision
+        mesh_filename="gripper/lite/collision/gripper_lite_finger"
+        origin_xyz="0 -0.0078 0.0543"
+        origin_rpy="0 0 0" />
+    </link>
+    <joint name="${prefix}right_finger_joint" type="prismatic">
+      <parent link="${prefix}lite_gripper_base_link"/>
+      <child link="${prefix}lite_gripper_right_finger"/>
+      <origin xyz="0 0 0" rpy="0 0 0"/>
+      <axis xyz="0 -1 0"/>
+      <limit lower="0.0" upper="0.0081" effort="2" velocity="0.1"/>
+    </joint>
+    <!-- TCP Link and Joint -->
     <link name="${prefix}link_tcp" />
     <joint name="${prefix}joint_tcp" type="fixed">
       <origin xyz="0 0 0.0836" rpy="0 0 0" />
-      <parent link="${prefix}uflite_gripper_link" />
+      <parent link="${prefix}lite_gripper_base_link" />
       <child link="${prefix}link_tcp" />
     </joint>

File: xarm_description/urdf/lite6/lite6.ros2_control.xacro (robot description, xacro)
@@ -11,20 +11,32 @@
     joint4_lower_limit:=${-2.0*pi}  joint4_upper_limit:=${2.0*pi}
     joint5_lower_limit:=${-2.1642}  joint5_upper_limit:=${2.1642}
-    joint6_lower_limit:=${-2.0*pi}  joint6_upper_limit:=${2.0*pi}">
+    joint6_lower_limit:=${-2.0*pi}  joint6_upper_limit:=${2.0*pi}
+    joint_commands_topic:='/isaac_joint_commands'
+    joint_states_topic:='/isaac_joint_states'">
     <ros2_control name="${prefix}${ros2_control_plugin}" type="system">
       <hardware>
-        <plugin>${ros2_control_plugin}</plugin>
-        <xacro:if value="${ros2_control_plugin == 'uf_robot_hardware/UFRobotSystemHardware'}">
-          <param name="hw_ns">${prefix}${hw_ns}</param>
-          <param name="velocity_control">${velocity_control}</param>
-          <param name="prefix">P${prefix}</param>
-          <param name="robot_ip">R${robot_ip}</param>
-          <param name="report_type">${report_type}</param>
-          <param name="dof">6</param>
-          <param name="baud_checkset">${baud_checkset}</param>
-          <param name="default_gripper_baud">${default_gripper_baud}</param>
-          <param name="robot_type">lite</param>
-          <param name="add_gripper">${add_gripper}</param>
+        <!-- Isaac special case: use a *token* 'isaac' to keep the node name valid -->
+        <xacro:if value="${ros2_control_plugin == 'isaac'}">
+          <plugin>topic_based_ros2_control/TopicBasedSystem</plugin>
+          <param name="joint_commands_topic">${joint_commands_topic}</param>
+          <param name="joint_states_topic">${joint_states_topic}</param>
         </xacro:if>
+        <!-- Everything else: behave like the original file -->
+        <xacro:unless value="${ros2_control_plugin == 'isaac'}">
+          <plugin>${ros2_control_plugin}</plugin>
+          <!-- Real xArm hardware parameters (only when that plugin is selected) -->
+          <xacro:if value="${ros2_control_plugin == 'uf_robot_hardware/UFRobotSystemHardware'}">
+            <param name="hw_ns">${prefix}${hw_ns}</param>
+            <param name="velocity_control">${velocity_control}</param>
+            <param name="prefix">P${prefix}</param>
+            <param name="robot_ip">R${robot_ip}</param>
+            <param name="report_type">${report_type}</param>
+            <param name="dof">6</param>
+            <param name="baud_checkset">${baud_checkset}</param>
+            <param name="default_gripper_baud">${default_gripper_baud}</param>
+            <param name="robot_type">lite</param>
+            <param name="add_gripper">${add_gripper}</param>
+          </xacro:if>
+        </xacro:unless>
       </hardware>
       <joint name="${prefix}joint1">

File: xarm_description/urdf/xarm_device_macro.xacro (robot description, xacro)
@@ -221,6 +221,7 @@
       <xacro:if value="${robot_type == 'lite'}">
         <!-- Load Lite Gripper Model URDF -->
-        <xacro:include filename="$(find xarm_description)/urdf/gripper/lite_gripper.urdf.xacro" />
-        <xacro:uflite_gripper_urdf prefix="${prefix}" attach_to="${prefix}link_eef" />
+        <xacro:include filename="$(find xarm_description)/urdf/gripper/lite_gripper_macro.xacro" />
+        <xacro:lite_gripper_macro prefix="${prefix}" attach_to="${prefix}link_eef"
+          ros2_control_plugin="${ros2_control_plugin}" dof="${dof}" hard_interface="${hard_interface}" />
       </xacro:if>
       <xacro:unless value="${robot_type == 'lite'}">

File: xarm_moveit_config/srdf/_lite6_macro.srdf.xacro (robot description, xacro)
@@ -43,18 +43,47 @@
       <joint name="${prefix}joint6" value="0" />
     </group_state>
+    <group_state name="hold-up" group="${prefix}lite6">
+      <joint name="${prefix}joint1" value="0" />
+      <joint name="${prefix}joint2" value="0" />
+      <joint name="${prefix}joint3" value="0" />
+      <joint name="${prefix}joint4" value="0" />
+      <joint name="${prefix}joint5" value="-1.5708" />
+      <joint name="${prefix}joint6" value="0" />
+    </group_state>
     <!-- gripper -->
     <xacro:if value="${add_gripper}">
-      <!-- <group name="${prefix}lite_gripper">
-        <joint name="${prefix}gripper_fix" />
-        <joint name="${prefix}joint_tcp" />
-      </group> -->
+      <group name="${prefix}lite_gripper">
+        <link name="${prefix}lite_gripper_base_link" />
+        <link name="${prefix}lite_gripper_left_finger" />
+        <link name="${prefix}lite_gripper_right_finger" />
+        <link name="${prefix}link_tcp" />
+        <joint name="${prefix}left_finger_joint" />
+        <joint name="${prefix}right_finger_joint" />
+      </group>
+      <group_state name="open" group="${prefix}lite_gripper">
+        <joint name="${prefix}left_finger_joint" value="0.0081" />
+        <joint name="${prefix}right_finger_joint" value="0.0081" />
+      </group_state>
+      <group_state name="close" group="${prefix}lite_gripper">
+        <joint name="${prefix}left_finger_joint" value="0" />
+        <joint name="${prefix}right_finger_joint" value="0" />
+      </group_state>
       <!-- END EFFECTOR, Purpose, Represent information about an end effector. -->
-      <!-- <end_effector name="${prefix}lite_gripper" parent_link="${prefix}link_tcp" group="${prefix}lite_gripper" /> -->
-      <passive_joint name="${prefix}gripper_fix" />
-      <!--PASSIVE JOINT, Purpose, this element is used to mark joints that are not actuated-->
+      <end_effector name="${prefix}lite_gripper" parent_link="${prefix}link_tcp" group="${prefix}lite_gripper" />
       <!-- DISABLE COLLISIONS, By default it is assumed that any link of the robot could potentially come into collision with any other link in the robot. This tag disables collision checking between a specified pair of links. -->
-      <disable_collisions link1="${prefix}link5" link2="${prefix}uflite_gripper_link" reason="Never" />
-      <disable_collisions link1="${prefix}link6" link2="${prefix}uflite_gripper_link" reason="Never" />
-      <disable_collisions link1="${prefix}link_eef" link2="${prefix}uflite_gripper_link" reason="Adjacent" />
+      <disable_collisions link1="${prefix}lite_gripper_left_finger" link2="${prefix}lite_gripper_base_link" reason="Adjacent" />
+      <disable_collisions link1="${prefix}lite_gripper_right_finger" link2="${prefix}lite_gripper_base_link" reason="Adjacent" />
+      <disable_collisions link1="${prefix}lite_gripper_left_finger" link2="${prefix}lite_gripper_right_finger" reason="Never" />
+      <disable_collisions link1="${prefix}lite_gripper_left_finger" link2="${prefix}link4" reason="Never" />
+      <disable_collisions link1="${prefix}lite_gripper_left_finger" link2="${prefix}link5" reason="Never" />
+      <disable_collisions link1="${prefix}lite_gripper_left_finger" link2="${prefix}link6" reason="Never" />
+      <disable_collisions link1="${prefix}lite_gripper_right_finger" link2="${prefix}link4" reason="Never" />
+      <disable_collisions link1="${prefix}lite_gripper_right_finger" link2="${prefix}link5" reason="Never" />
+      <disable_collisions link1="${prefix}lite_gripper_right_finger" link2="${prefix}link6" reason="Never" />
+      <disable_collisions link1="${prefix}link6" link2="${prefix}lite_gripper_base_link" reason="Adjacent" />
+      <disable_collisions link1="${prefix}link5" link2="${prefix}lite_gripper_base_link" reason="Never" />
+      <disable_collisions link1="${prefix}link_eef" link2="${prefix}lite_gripper_left_finger" reason="Never" />
+      <disable_collisions link1="${prefix}link_eef" link2="${prefix}lite_gripper_right_finger" reason="Never" />
+      <disable_collisions link1="${prefix}link_eef" link2="${prefix}lite_gripper_base_link" reason="Adjacent" />
     </xacro:if>
     <!-- vacuum gripper -->
