Commit message: updates to enable lite gripper in Isaac SIM

File: xarm_description/urdf/gripper/lite_gripper.ros2_control.xacro (robot description, xacro)
@@ -5,5 +5,5 @@
       prefix:=''
       ros2_control_plugin:=''
-      isaac_cmd_topic:='/isaac_joint_commands'
+      isaac_cmd_topic:='/isaac_joint_commands_gripper'
       isaac_state_topic:='/isaac_joint_states'
     ">

File: xarm_description/urdf/gripper/lite_gripper.urdf.xacro (robot description, xacro)
@@ -53,5 +53,5 @@
       <child link="${prefix}lite_gripper_left_finger"/>
       <axis xyz="0 1 0"/>
-      <limit lower="0.0" upper="0.0081" effort="2" velocity="0.1"/>
+      <limit lower="0.0" upper="0.0081" effort="10000" velocity="0.1"/>
       <mimic joint="${prefix}right_finger_joint" multiplier="1" offset="0" />
     </joint>
@@ -80,5 +80,5 @@
       <origin xyz="0 0 0" rpy="0 0 0"/>
       <axis xyz="0 -1 0"/>
-      <limit lower="0.0" upper="0.0081" effort="2" velocity="0.1"/>
+      <limit lower="0.0" upper="0.0081" effort="10000" velocity="0.1"/>
     </joint>
     <!-- TCP Link and Joint -->
