Commit message: updated to enable interaction with Isaac SIM

File: xarm_description/urdf/gripper/lite_gripper.urdf.xacro (robot description, xacro)
@@ -1,13 +1,15 @@
 <?xml version="1.0"?>
-<robot xmlns:xacro="http://ros.org/wiki/xacro" name="uflite_gripper">
-  <xacro:macro name="uflite_gripper_urdf" params="prefix:='' attach_to:='' attach_xyz:='0 0 0' attach_rpy:='0 0 0' ">
+<robot xmlns:xacro="http://ros.org/wiki/xacro" name="uf_lite_gripper">
+  <xacro:macro name="lite_gripper_urdf" params="prefix:='' attach_to:='' attach_xyz:='0 0 0' attach_rpy:='0 0 0' ">
+    <!-- Gripper Fix Joint -->
     <xacro:unless value="${attach_to == ''}">
       <joint name="${prefix}gripper_fix" type="fixed">
         <parent link="${attach_to}"/>
-        <child link="${prefix}uflite_gripper_link"/>
+        <child link="${prefix}lite_gripper_base_link"/>
         <origin xyz="${attach_xyz}" rpy="${attach_rpy}"/>
       </joint>
     </xacro:unless>
-    <link name="${prefix}uflite_gripper_link">
+    <!-- Base link of the gripper -->
+    <link name="${prefix}lite_gripper_base_link">
       <inertial>
         <origin xyz="0.0 0.0 0.030" rpy="0 0 0" />
@@ -18,17 +20,71 @@
       </inertial>
       <xacro:common_link_visual
-        mesh_filename="gripper/lite/visual/gripper_lite"
+        mesh_filename="gripper/lite/visual/gripper_lite_body"
         origin_xyz="0 0 0"
         origin_rpy="0 0 0"
         material_name="${prefix}White" />
       <xacro:common_link_collision
-        mesh_filename="gripper/lite/collision/gripper_lite"
+        mesh_filename="gripper/lite/collision/gripper_lite_body"
         origin_xyz="0 0 0"
         origin_rpy="0 0 0" />
     </link>
+    <!-- Left Finger -->
+    <link name="${prefix}lite_gripper_left_finger">
+      <inertial>
+        <origin xyz="0 0.0078 0.0543" rpy="0 0 0" />
+        <mass value="0.012105" />
+        <inertia
+          ixx="3.7322E-06" ixy="-4.1705E-06" ixz="4.0142E-06"
+          iyy="1.744E-05" iyz="-1.2237E-06" izz="1.7775E-05" />
+      </inertial>
+      <xacro:common_link_visual
+        mesh_filename="gripper/lite/visual/gripper_lite_finger"
+        origin_xyz="0 0.0078 0.0543"
+        origin_rpy="0 0 3.14159"
+        material_name="${prefix}White" />
+      <xacro:common_link_collision
+        mesh_filename="gripper/lite/collision/gripper_lite_finger"
+        origin_xyz="0 0.0078 0.0543"
+        origin_rpy="0 0 3.14159" />
+    </link>
+    <joint name="${prefix}left_finger_joint" type="prismatic">
+      <origin xyz="0 0 0" rpy="0 0 0"/>
+      <parent link="${prefix}lite_gripper_base_link"/>
+      <child link="${prefix}lite_gripper_left_finger"/>
+      <axis xyz="0 1 0"/>
+      <limit lower="0.0" upper="0.0081" effort="10000" velocity="0.1"/>
+      <mimic joint="${prefix}right_finger_joint" multiplier="1" offset="0" />
+    </joint>
+    <!-- Right Finger -->
+    <link name="${prefix}lite_gripper_right_finger">
+      <inertial>
+        <origin xyz="0 -0.0078 0.0543" rpy="0 0 0" />
+        <mass value="0.012068" />
+        <inertia
+          ixx="4.1413E-06" ixy="3.9682E-06" ixz="4.5734E-06"
+          iyy="1.6115E-05" iyz="1.6711E-06" izz="1.6032E-05" />
+      </inertial>
+      <xacro:common_link_visual
+        mesh_filename="gripper/lite/visual/gripper_lite_finger"
+        origin_xyz="0 -0.0078 0.0543"
+        origin_rpy="0 0 0"
+        material_name="${prefix}White" />
+      <xacro:common_link_collision
+        mesh_filename="gripper/lite/collision/gripper_lite_finger"
+        origin_xyz="0 -0.0078 0.0543"
+        origin_rpy="0 0 0" />
+    </link>
+    <joint name="${prefix}right_finger_joint" type="prismatic">
+      <parent link="${prefix}lite_gripper_base_link"/>
+      <child link="${prefix}lite_gripper_right_finger"/>
+      <origin xyz="0 0 0" rpy="0 0 0"/>
+      <axis xyz="0 -1 0"/>
+      <limit lower="0.0" upper="0.0081" effort="10000" velocity="0.1"/>
+    </joint>
+    <!-- TCP Link and Joint -->
     <link name="${prefix}link_tcp" />
     <joint name="${prefix}joint_tcp" type="fixed">
       <origin xyz="0 0 0.0836" rpy="0 0 0" />
-      <parent link="${prefix}uflite_gripper_link" />
+      <parent link="${prefix}lite_gripper_base_link" />
       <child link="${prefix}link_tcp" />
     </joint>

File: xarm_description/urdf/xarm_device_macro.xacro (robot description, xacro)
@@ -52,9 +52,9 @@
     <!-- Specify Mesh file path -->
     <xacro:property name="mesh_suffix" value="${mesh_suffix}" scope="parent"/>
-    <xacro:if value="${ros2_control_plugin == 'gazebo_ros2_control/GazeboSystem' or ros2_control_plugin == 'ign_ros2_control/IgnitionSystem' or ros2_control_plugin == 'gz_ros2_control/GazeboSimSystem'}">
+    <xacro:if value="${ros2_control_plugin == 'gazebo_ros2_control/GazeboSystem' or ros2_control_plugin == 'ign_ros2_control/IgnitionSystem'}">
       <!-- gazebo use -->
       <xacro:property name="mesh_path" value="file://$(find xarm_description)/meshes" scope="parent"/>
     </xacro:if>
-    <xacro:unless value="${ros2_control_plugin == 'gazebo_ros2_control/GazeboSystem' or ros2_control_plugin == 'ign_ros2_control/IgnitionSystem' or ros2_control_plugin == 'gz_ros2_control/GazeboSimSystem'}">
+    <xacro:unless value="${ros2_control_plugin == 'gazebo_ros2_control/GazeboSystem' or ros2_control_plugin == 'ign_ros2_control/IgnitionSystem'}">
       <xacro:property name="mesh_path" value="package://xarm_description/meshes" scope="parent"/>
     </xacro:unless>
@@ -221,6 +221,7 @@
       <xacro:if value="${robot_type == 'lite'}">
         <!-- Load Lite Gripper Model URDF -->
-        <xacro:include filename="$(find xarm_description)/urdf/gripper/lite_gripper.urdf.xacro" />
-        <xacro:uflite_gripper_urdf prefix="${prefix}" attach_to="${prefix}link_eef" />
+        <xacro:include filename="$(find xarm_description)/urdf/gripper/lite_gripper_macro.xacro" />
+        <xacro:lite_gripper_macro prefix="${prefix}" attach_to="${prefix}link_eef"
+          ros2_control_plugin="${ros2_control_plugin}" dof="${dof}" hard_interface="${hard_interface}" />
       </xacro:if>
       <xacro:unless value="${robot_type == 'lite'}">
